File: LinkPlug-RS422.kicad_sch (KiCad schematic)
At the start: 8 parts, among them J2001 2x05_Horizontal, U301 LTC2863

Commit message: Update to Kicad 8
Parts:
- renumbered TP102 to TP301, TP102 to TP302, TP102 to TP303, TP102 to TP304
